Commit message: adding training functionality for cartpole. modified cartpoleslide bot to start in stable equilibrium

File: urdf/cartpoleslide.urdf.xacro (robot description, xacro)
@@ -49,5 +49,5 @@
             </material>
         </visual>
-        <collision>
+        <!-- <collision>
             <origin xyz="0 0 ${l_rod/2+t_cart/2}" rpy = "0 0 0"/>
             <geometry>
@@ -57,5 +57,5 @@
                 <color rgba="1 1 1 1"/>
             </material>
-        </collision>
+        </collision> -->
         <inertial>
             <origin xyz="0 0 ${l_rod/2+t_cart/2}" rpy="0 0 0"/>
@@ -74,5 +74,5 @@
             </material>
         </visual>
-        <collision>
+        <!-- <collision>
             <origin xyz="0 0 0" rpy = "0 0 0"/>
             <geometry>
@@ -82,5 +82,5 @@
                 <color rgba="1 1 1 1"/>
             </material>
-        </collision>
+        </collision> -->
         <inertial>
             <origin xyz="0 0 0" rpy="0 0 0"/>
@@ -95,9 +95,9 @@
         <axis xyz="0 0 0"/>
     </joint>
-    <joint name="pole_joint" type="revolute">
-        <limit lower="-0.78" upper="0.78" effort="1000.0" velocity="10000.0"/>
+    <joint name="pole_joint" type="continuous">
+        <!-- <limit lower="-0.78" upper="0.78" effort="1000.0" velocity="10000.0"/> -->
         <parent link="platform"/>
         <child link="rod"/>
-        <origin xyz="0 0 0" rpy="0 0 0"/>
+        <origin xyz="0 0 0" rpy="0 3.141 0"/>
         <axis xyz="0 1 0"/>
     </joint>

Commit message: linear turtlebot koopman test, improved cartpole estimation

File: urdf/cartpoleslide.urdf.xacro (robot description, xacro)
@@ -99,5 +99,5 @@
         <parent link="platform"/>
         <child link="rod"/>
-        <origin xyz="0 0 0" rpy="0 3.141 0"/>
+        <origin xyz="0 0 0" rpy="0 2.356 0"/>
         <axis xyz="0 1 0"/>
     </joint>
